Commit message: for search problems

File: simple_dog_simulation/simpledog/urdf/laikago/gazebo.xacro (robot description, xacro)
@@ -30,14 +30,14 @@
     </gazebo>
     <!-- Show the trajectory of foot. You can add another trajectory about another foot. -->
-    <!-- <gazebo>
+    <gazebo>
         <plugin name="3dplot" filename="libLinkPlot3DPlugin.so">
             <frequency>100</frequency>
             <plot>
-                <link>FL_foot</link>
+                <link>LF_FOOT</link>
                 <pose>0 0 0 0 0 0</pose>
                 <material>Gazebo/Green</material>
             </plot>
         </plugin>
-    </gazebo> -->
+    </gazebo>
     <gazebo>
         <plugin filename="libgazebo_ros_force.so" name="gazebo_ros_force">
