Commit message: Golaoxu : Init WBC

File: simple_dog_simulation/simpledog/urdf/laikago/my_laika.xacro (robot description, xacro)
@@ -16,4 +16,10 @@
         </joint>
     </xacro:if>
+    <!-- <link name="world"/>
+    <joint name="base_static_joint1" type="fixed">
+        <origin rpy="0 0 0" xyz="0 0 1"/>
+        <parent link="world"/>
+        <child link="base"/>
+    </joint> -->
     <link name="base">
         <visual>
